Commit message: 修正urdf两腿重量不一致

File: source/oceanisaaclab/assets/urdf/ocean.urdf (robot description, URDF)
Before this commit: robot ocean, 16 links, 15 joints
Links:
- link leg_l1_link: mass 0.33145 -> 0.33146
- link leg_l2_link: mass 0.12555 -> 0.15568
- link leg_l4_link: mass 0.4525 -> 0.45582
- link leg_l5_link: mass 0.39976 -> 0.45151
